File: STM32F030F4_devboard.kicad_pcb (KiCad board)
At the start: 2 copper layers, 28 parts, among them J1 USB_B_Micro, J2 Conn_01x04_Pin, J3 Conn_01x07_Pin, J4 Conn_01x07_Pin, J5 Conn_01x03_Pin, SW2 SW_Push, U1 STM32F030F4P6, U2 AMS1117-3.3, Y1 24Mhz

Commit message: finish pcb routing
Parts:
- added H1: MountingHole, MountingHole:MountingHole_2.2mm_M2, F.Cu at (136.0, 144.0)
- added H2: MountingHole, MountingHole:MountingHole_2.2mm_M2, F.Cu at (136.0, 123.0)
- added H3: MountingHole, MountingHole:MountingHole_2.2mm_M2, F.Cu at (95.0, 144.0)
- added H4: MountingHole, MountingHole:MountingHole_2.2mm_M2, F.Cu at (95.0, 123.0)
- added J6: Conn_01x03_Pin, Connector_PinHeader_2.54mm:PinHeader_1x03_P2.54mm_Vertical, F.Cu at (112.0, 145.0)
- J3, J4: value Conn_01x07_Pin -> Conn_01x04_Pin; footprint Connector_PinHeader_2.54mm:PinHeader_1x07_P2.54mm_Vertical -> Connector_PinHeader_2.54mm:PinHeader_1x04_P2.54mm_Vertical
- SW2: footprint Button_Switch_SMD:SW_Push_1P1T_NO_6x6mm_H9.5mm -> Button_Switch_SMD:SW_SPST_PTS645
- moved J5 110.7 mm to (94.6, 137.7), turned to 180 degrees
- moved R1 93.6 mm to (97.3, 134.1), turned to 90 degrees
- moved J3 92.0 mm to (100.6, 145.0), turned to 90 degrees
- moved R7 86.5 mm to (105.8, 128.2)
- moved R6 86.1 mm to (116.1, 137.1)
- moved D2 83.5 mm to (119.5, 137.1)
- moved D1 80.9 mm to (122.6, 134.2), turned to 90 degrees
- moved C9 78.3 mm to (127.5, 137.2), turned to 180 degrees
- moved SW2 76.6 mm to (102.8, 123.8)
- moved C11 75.5 mm to (109.2, 128.2)
- moved R2 74.9 mm to (123.4, 137.2)
- moved C10 74.2 mm to (122.6, 130.6), turned to -90 degrees
- moved R3 65.1 mm to (123.0, 125.5), turned to 180 degrees
- moved R4 60.2 mm to (127.3, 125.6)
- moved J4 60.0 mm to (129.1, 122.9), turned to -90 degrees
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Connections:
- net Net-(U1-PB1) renamed /user_led
- J3 pad 1: /MISO -> Net-(J3-Pin_1)
- J3 pad 2: /SCLK -> /USART_RX
- J3 pad 3: Net-(J3-Pin_3) -> /USART_TX
- J3 pad 4: /USART_RX -> Net-(J3-Pin_4)
- J4 pad 2: +3.3V -> /SCL
- J4 pad 3: GND -> /SDA
- R3 pad 1: +3.3V -> /SDA
- R3 pad 2: /SDA -> +3.3V
- R4 pad 1: +3.3V -> /SCL
- R4 pad 2: /SCL -> +3.3V
- R5 pad 1: +3.3VA -> +3.3V
- R5 pad 2: +3.3V -> +3.3VA
- U1 pad 10: Net-(J3-Pin_3) -> Net-(J3-Pin_1)
- U1 pad 6: Net-(J3-Pin_7) -> unconnected-(U1-PA0-Pad6)
- U1 pad 7: Net-(J3-Pin_6) -> Net-(J3-Pin_4)
- Y1 pad 2: Net-(Y1-Pad2) -> GND
- Y1 pad 4: Net-(Y1-Pad2) -> GND
Routing:
- net +3.3V: track 0.00 -> 109.6 mm, vias 0 -> 2
- net GND: track 0.00 -> 33.9 mm, vias 0 -> 20
- net /SCL: track 0.00 -> 19.1 mm
- net /SDA: track 0.00 -> 17.0 mm
- net /BOOT0: track 0.00 -> 14.1 mm
- net Net-(J3-Pin_4): track 0.00 -> 13.7 mm
- net Net-(J3-Pin_1): track 0.00 -> 13.6 mm
- net /USART_RX: track 0.00 -> 13.4 mm
- net /MISO: track 0.00 -> 13.2 mm
- net /USART_TX: track 0.00 -> 13.2 mm
- net /NRST: track 0.00 -> 12.6 mm
- net /MOSI: track 0.00 -> 12.6 mm
- net /SCLK: track 0.00 -> 10.3 mm
- net +3.3VA: track 0.00 -> 9.78 mm
- net /SWDIO: track 0.00 -> 9.37 mm
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- added copper zone on F.Cu, net +3.3V
- added copper zone on B.Cu, net GND
- added copper zone on F.Cu, net GND
- added copper zone on F.Cu, net VBUS
Other:
- board outline added: 47 x 27 mm
- board text added: "3.3"
- board text added: "MISO"
- board text added: "MOSI"
- board text added: "RX"
- board text added: "SCLK"
- board text added: "TX"
- board text added: "boot"
- board text added: "pb1_led"
- board text added: "pwr"
- board text added: "reset"
- board text added: "scl"
- board text added: "swclk"
- board text added: "swdio"
