File: STM32F030F4_devboard.kicad_sch (KiCad schematic)
At the start: 28 parts, among them J1 USB_B_Micro, J2 Conn_01x04_Pin, J3 Conn_01x07_Pin, J4 Conn_01x07_Pin, J5 Conn_01x03_Pin, SW2 SW_Push, U1 STM32F030F4P6, U2 AMS1117-3.3, Y1 24Mhz

Commit message: finish pcb routing
Parts:
- removed J3, J4: Conn_01x07_Pin, Connector_PinHeader_2.54mm:PinHeader_1x07_P2.54mm_Vertical, symbol Connector:Conn_01x07_Pin
- added H1, H2, H3, H4: MountingHole, MountingHole:MountingHole_2.2mm_M2, symbol Mechanical:MountingHole
- added J3, J4: Conn_01x04_Pin, Connector_PinHeader_2.54mm:PinHeader_1x04_P2.54mm_Vertical, symbol Connector:Conn_01x04_Pin
- added J6: Conn_01x03_Pin, Connector_PinHeader_2.54mm:PinHeader_1x03_P2.54mm_Vertical, symbol Connector:Conn_01x03_Pin
Connections:
- net +3.3V: now also R3.2, R4.2, R5.1, J4.1 (Pin_1); no longer R3.1, R4.1, R5.2
- net +3.3VA: now also R5.2; no longer R5.1
- net GND: now also Y1.2, Y1.4, J4.4 (Pin_4)
- net MISO: now also J6.2 (Pin_2)
- net MOSI: now also J6.1 (Pin_1)
- net SCL: now also R4.1, J4.2 (Pin_2); no longer R4.2
- net SCLK: now also J6.3 (Pin_3)
- net SDA: now also R3.1, J4.3 (Pin_3); no longer R3.2
- net USART_RX: now also J3.2 (Pin_2)
- net USART_TX: now also J3.3 (Pin_3)
- net user_led: now reaches R6.1, U1.14 (PB1)
- net at U1.10 (PA4): now also J3.1 (Pin_1)
- net at U1.7 (PA1): now also J3.4 (Pin_4)
- no-connect marks 4 -> 5
Other:
- note added: "mounting hole"
- moved on the sheet: D2, R5, R6
